Commit message: feat: add ros2 control

File: description/gazebo_control.xacro (robot description, xacro)
@@ -5,6 +5,6 @@
             <left_joint>left_wheel_joint</left_joint>
             <right_joint>right_wheel_joint</right_joint>
-            <right_joint>right_wheel_joint</right_joint>
             <right_joint>wheel_back_right_joint</right_joint>
+            <left_joint>wheel_back_left_joint</left_joint>
             <wheel_separation>1.8</wheel_separation>
             <wheel_radius>0.25</wheel_radius>

File: description/robot.urdf.xacro (robot description, xacro)
@@ -1,4 +1,6 @@
 <?xml version="1.0"?>
 <robot xmlns:xacro="http://www.ros.org/wiki/xacro"  name="robot">
+    <xacro:arg name="use_ros2_control" default="true"/>
+    <!-- <xacro:arg name="type_leg_joint" defaut="revolute"/> -->
     <xacro:include filename="robot_core_control.xacro" />
     <xacro:include filename="lidar.xacro" />
@@ -6,5 +8,10 @@
     <xacro:include filename="imu.xacro" />
     <xacro:include filename="gps.xacro" />
-    <!-- <xacro:include filename="ros2_control.xacro" /> -->
-    <xacro:include filename="gazebo_control.xacro" />
+    <!-- <xacro:include filename="gazebo_control.xacro" /> -->
+    <xacro:if value="$(arg use_ros2_control)">
+        <xacro:include filename="ros2_control.xacro" />
+    </xacro:if>
+    <xacro:unless value="$(arg use_ros2_control)">
+        <xacro:include filename="gazebo_control.xacro" />
+    </xacro:unless>
 </robot>

File: description/robot_core_control.xacro (robot description, xacro)
@@ -70,5 +70,5 @@
         <disable_collision>1</disable_collision>
     </joint>
-    <joint name="left_wheel_leg_joint" type="fixed">  <!-- revolute to ros2 control -->
+    <joint name="left_wheel_leg_joint" type="revolute">  <!-- revolute to ros2 control and fixed to diffdrive -->
         <parent link="base_link"/>
         <child link="left_leg_link"/>
@@ -118,5 +118,5 @@
         <disable_collision>0</disable_collision>
     </joint>
-    <joint name="right_wheel_leg_joint" type="fixed">   <!-- revolute to ros2 control -->
+    <joint name="right_wheel_leg_joint" type="revolute">   <!-- revolute to ros2 control and fixed to diffdrive -->
         <parent link="base_link"/>
         <child link="right_leg_link"/>
@@ -166,5 +166,5 @@
     <disable_collision>0</disable_collision>
 </joint>
-<joint name="right_wheel_back_leg_joint" type="fixed">  <!-- revolute to ros2 control -->
+<joint name="right_wheel_back_leg_joint" type="revolute">  <!-- revolute to ros2 control and fixed to diffdrive  -->
         <parent link="base_link"/>
         <child link="right_back_leg_link"/>
@@ -214,5 +214,5 @@
     <disable_collision>0</disable_collision>
 </joint>
-<joint name="left_wheel_back_leg_joint" type="fixed"> <!-- revolute to ros2 control -->
+<joint name="left_wheel_back_leg_joint" type="revolute"> <!-- revolute to ros2 control and fixed to diffdrive -->
         <parent link="base_link"/>
         <child link="left_back_leg_link"/>

File: description/ros2_control.xacro (robot description, xacro)
@@ -21,4 +21,20 @@
             <state_interface name="position"/>
         </joint>
+        <joint name="wheel_back_right_joint">
+            <command_interface name="velocity">
+                <param name="min">-10</param>
+                <param name="max">10</param>
+            </command_interface>
+            <state_interface name="velocity"/>
+            <state_interface name="position"/>
+        </joint>
+        <joint name="wheel_back_left_joint">
+            <command_interface name="velocity">
+                <param name="min">-10</param>
+                <param name="max">10</param>
+            </command_interface>
+            <state_interface name="velocity"/>
+            <state_interface name="position"/>
+        </joint>
     </ros2_control>
     <gazebo>
@@ -26,6 +42,6 @@
             <robot_param>robot_description</robot_param>
             <robot_param_node>robot_state_publisher</robot_param_node>
-            <parameters>$(find gzmy_bot)/config/my_controllers.yaml</parameters>
-            <parameters>$(find gzmy_bot)/config/gaz_ros2_ctl_use_sim.yaml</parameters>
+            <parameters>$(find base_desc)/config/my_controllers.yaml</parameters>
+            <parameters>$(find base_desc)/config/gaz_ros2_ctl_use_sim.yaml</parameters>
         </plugin>
     </gazebo>
