Commit message: feat: diff drive controller

File: description/robot_core_control.xacro (robot description, xacro)
@@ -70,5 +70,5 @@
         <disable_collision>1</disable_collision>
     </joint>
-    <joint name="left_wheel_leg_joint" type="revolute">  <!-- revolute to ros2 control and fixed to diffdrive -->
+    <joint name="left_wheel_leg_joint" type="fixed">  <!-- revolute to ros2 control and fixed to diffdrive -->
         <parent link="base_link"/>
         <child link="left_leg_link"/>
@@ -118,5 +118,5 @@
         <disable_collision>0</disable_collision>
     </joint>
-    <joint name="right_wheel_leg_joint" type="revolute">   <!-- revolute to ros2 control and fixed to diffdrive -->
+    <joint name="right_wheel_leg_joint" type="fixed">   <!-- revolute to ros2 control and fixed to diffdrive -->
         <parent link="base_link"/>
         <child link="right_leg_link"/>
@@ -166,5 +166,5 @@
     <disable_collision>0</disable_collision>
 </joint>
-<joint name="right_wheel_back_leg_joint" type="revolute">  <!-- revolute to ros2 control and fixed to diffdrive  -->
+<joint name="right_wheel_back_leg_joint" type="fixed">  <!-- revolute to ros2 control and fixed to diffdrive  -->
         <parent link="base_link"/>
         <child link="right_back_leg_link"/>
@@ -214,5 +214,5 @@
     <disable_collision>0</disable_collision>
 </joint>
-<joint name="left_wheel_back_leg_joint" type="revolute"> <!-- revolute to ros2 control and fixed to diffdrive -->
+<joint name="left_wheel_back_leg_joint" type="fixed"> <!-- revolute to ros2 control and fixed to diffdrive -->
         <parent link="base_link"/>
         <child link="left_back_leg_link"/>
