Commit message: feat: add camera like realsense

File: faucon_base_desc/description_mini/camera.xacro (robot description, xacro)
@@ -24,28 +24,38 @@
         <parent link="camera_link"/>
         <child link="camera_link_optical"/>
-        <origin xyz="0 0 0" rpy="${-pi/2} 0 ${-pi/2}"/>
+        <origin xyz="0 0 0.161" rpy="0.0 0 0.0"/>
     </joint>
     <link name="camera_link_optical"></link>
     <gazebo reference="camera_link">
         <material>Gazebo/Black</material>
-        <sensor name="camera" type="camera">
-            <pose> 0 0 0 0 0 0 </pose>
-            <visualize>true</visualize>
-            <update_rate>10</update_rate>
+        <sensor name="rgbd_camera" type="rgbd_camera">
+            <update_rate>20</update_rate>
+            <topic>depth_camera</topic>
+            <gz_frame_id>camera_link_optical</gz_frame_id>
             <camera>
-                <camera_info_topic>camera/camera_info</camera_info_topic>
                 <horizontal_fov>1.089</horizontal_fov>
                 <image>
-                    <format>R8G8B8</format>
                     <width>640</width>
                     <height>480</height>
+                    <format>RGB_INT8</format>
                 </image>
                 <clip>
                     <near>0.05</near>
-                    <far>8.0</far>
+                    <far>10.0</far>
                 </clip>
             </camera>
-            <topic>camera/image_raw</topic>
-            <gz_frame_id>camera_link_optical</gz_frame_id>
+            <depth_camera>
+                <clip>
+                    <near>0.05</near>
+                    <far>10.0</far>
+                </clip>
+                <noise>
+                    <type>gaussian</type>
+                    <mean>0.0</mean>
+                    <stddev>0.001</stddev>
+                </noise>
+            </depth_camera>
+            <always_on>1</always_on>
+            <visualize>true</visualize>
         </sensor>
     </gazebo>

Commit message: change frame gazebo point cloud

File: faucon_base_desc/description_mini/camera.xacro (robot description, xacro)
@@ -4,5 +4,5 @@
         <parent link="chassis"/>
         <child link="camera_link"/>
-        <origin xyz="0.142 0 0.161" rpy="0 0 0"/>
+        <origin xyz="0.142 0 0.138" rpy="0 0 0"/>
     </joint>
     <link name="camera_link">
@@ -24,5 +24,5 @@
         <parent link="camera_link"/>
         <child link="camera_link_optical"/>
-        <origin xyz="0 0 0.161" rpy="0.0 0 0.0"/>
+        <origin xyz="0 0 0" rpy="${-pi/2} 0 ${-pi/2}"/>
     </joint>
     <link name="camera_link_optical"></link>
@@ -32,5 +32,5 @@
             <update_rate>20</update_rate>
             <topic>depth_camera</topic>
-            <gz_frame_id>camera_link_optical</gz_frame_id>
+            <gz_frame_id>camera_link</gz_frame_id>
             <camera>
                 <horizontal_fov>1.089</horizontal_fov>

File: faucon_base_desc/description_mini/gps.xacro (robot description, xacro)
@@ -1,46 +1,24 @@
 <?xml version="1.0"?>
 <robot xmlns:xacro="http://www.ros.org/wiki/xacro">
-  <!-- Joint fixe entre le châssis et le GNSS -->
   <joint name="gnss_joint" type="fixed">
     <parent link="chassis"/>
     <child link="gnss_frame"/>
-    <!-- Positionne le GNSS (exemple au-dessus du châssis) -->
     <origin xyz="0.10 0 0.80" rpy="0 0 0"/>
   </joint>
-  <!-- Lien du capteur GNSS (petit cylindre pour le visuel) -->
   <link name="gnss_frame">
-    <!-- <visual>
-      <geometry>
-        <cylinder radius="0.03" length="0.02"/>
-      </geometry>
-      <material name="black"/>
-    </visual>
-    <collision>
-      <geometry>
-        <cylinder radius="0.03" length="0.02"/>
-      </geometry>
-    </collision>
-    <xacro:inertial_cylinder mass="0.05" length="0.02" radius="0.03">
-      <origin xyz="0 0 0" rpy="0 0 0"/>
-    </xacro:inertial_cylinder> -->
   </link>
-  <!-- Définition du capteur GNSS pour Gazebo Sim -->
   <gazebo reference="gnss_frame">
     <material>Gazebo/Black</material>
-    <!-- Capteur GNSS -->
     <sensor name="gnss" type="navsat">
       <pose>0 0 0 0 0 0</pose>
-      <!-- topic côté Gazebo ; tu peux changer -->
       <topic>/gnss/fix</topic>
-      <!-- Frame publiée (utile pour le bridge ROS2) -->
       <gz_frame_id>gnss_frame</gz_frame_id>
       <update_rate>10</update_rate>
       <navsat>
-        <!-- Modèle de bruit simple ; ajuste à ta convenance -->
         <position_sensing>
           <horizontal>
             <noise type="gaussian">
               <mean>0.0</mean>
-              <stddev>0.5</stddev>      <!-- ~0.5 m -->
+              <stddev>0.0001</stddev>
             </noise>
           </horizontal>
@@ -48,5 +26,5 @@
             <noise type="gaussian">
               <mean>0.0</mean>
-              <stddev>1.0</stddev>      <!-- ~1.0 m -->
+              <stddev>0.0001</stddev>
             </noise>
           </vertical>
@@ -55,9 +33,8 @@
           <noise type="gaussian">
             <mean>0.0</mean>
-            <stddev>0.1</stddev>        <!-- optionnel -->
+            <stddev>0.0001</stddev>
           </noise>
         </velocity_sensing>
       </navsat>
-      <!-- Affichage dans l’UI de Gazebo (facultatif) -->
       <visualize>true</visualize>
     </sensor>
