Commit message: feat: 04ws control

File: faucon_base_desc/description/robot_core_control.xacro (robot description, xacro)
@@ -70,5 +70,5 @@
         <disable_collision>1</disable_collision>
     </joint>
-    <joint name="left_wheel_leg_joint" type="fixed">  <!-- revolute to ros2 control and fixed to diffdrive -->
+    <joint name="left_wheel_leg_joint" type="revolute">  <!-- revolute to ros2 control and fixed to diffdrive -->
         <parent link="base_link"/>
         <child link="left_leg_link"/>
@@ -118,5 +118,5 @@
         <disable_collision>0</disable_collision>
     </joint>
-    <joint name="right_wheel_leg_joint" type="fixed">   <!-- revolute to ros2 control and fixed to diffdrive -->
+    <joint name="right_wheel_leg_joint" type="revolute">   <!-- revolute to ros2 control and fixed to diffdrive -->
         <parent link="base_link"/>
         <child link="right_leg_link"/>
@@ -166,5 +166,5 @@
     <disable_collision>0</disable_collision>
 </joint>
-<joint name="right_wheel_back_leg_joint" type="fixed">  <!-- revolute to ros2 control and fixed to diffdrive  -->
+<joint name="right_wheel_back_leg_joint" type="revolute">  <!-- revolute to ros2 control and fixed to diffdrive  -->
         <parent link="base_link"/>
         <child link="right_back_leg_link"/>
@@ -214,5 +214,5 @@
     <disable_collision>0</disable_collision>
 </joint>
-<joint name="left_wheel_back_leg_joint" type="fixed"> <!-- revolute to ros2 control and fixed to diffdrive -->
+<joint name="left_wheel_back_leg_joint" type="revolute"> <!-- revolute to ros2 control and fixed to diffdrive -->
         <parent link="base_link"/>
         <child link="left_back_leg_link"/>

File: faucon_base_desc/description/ros2_control.xacro (robot description, xacro)
@@ -37,4 +37,36 @@
             <state_interface name="position"/>
         </joint>
+        <joint name="right_wheel_back_leg_joint">
+            <command_interface name="position">
+                <param name="min">-10</param>
+                <param name="max">10</param>
+            </command_interface>
+            <state_interface name="velocity"/>
+            <state_interface name="position"/>
+        </joint>
+        <joint name="left_wheel_back_leg_joint">
+            <command_interface name="position">
+                <param name="min">-10</param>
+                <param name="max">10</param>
+            </command_interface>
+            <state_interface name="velocity"/>
+            <state_interface name="position"/>
+        </joint>
+        <joint name="right_wheel_leg_joint">
+            <command_interface name="position">
+                <param name="min">-10</param>
+                <param name="max">10</param>
+            </command_interface>
+            <state_interface name="velocity"/>
+            <state_interface name="position"/>
+        </joint>
+        <joint name="left_wheel_leg_joint">
+            <command_interface name="position">
+                <param name="min">-10</param>
+                <param name="max">10</param>
+            </command_interface>
+            <state_interface name="velocity"/>
+            <state_interface name="position"/>
+        </joint>
     </ros2_control>
     <gazebo>
@@ -42,5 +74,5 @@
             <robot_param>robot_description</robot_param>
             <robot_param_node>robot_state_publisher</robot_param_node>
-            <parameters>$(find faucon_base_desc)/config/my_controllers.yaml</parameters>
+            <parameters>$(find faucon_base_desc)/config/steer_controllers.yaml</parameters>
             <parameters>$(find faucon_base_desc)/config/gaz_ros2_ctl_use_sim.yaml</parameters>
         </plugin>

Commit message: some refactor

File: faucon_base_desc/description/robot_core_control.xacro (robot description, xacro)
@@ -19,4 +19,5 @@
     <xacro:property name="wheel_offset_y" value="0.5"/>
     <xacro:property name="wheel_offset_z" value="0.01"/>
+    <xacro:property name="caster_wheel_radius" value="0.12"/>
     <xacro:property name="caster_wheel_offset_x" value="0.350"/>
     <xacro:property name="caster_wheel_offset_z" value="${wheel_offset_z - wheel_radius + caster_wheel_radius}"/>
