Commit message: move the origin from rear to center

File: faucon_base_desc/description/camera.xacro (robot description, xacro)
@@ -4,5 +4,5 @@
         <parent link="base_link"/>
         <child link="camera_link"/>
-        <origin xyz="1.3 0.0 0.3" rpy="0.0 0.33 0"/>
+        <origin xyz="0.65 0.0 0.3" rpy="0.0 0.33 0"/>
     </joint>
     <link name="camera_link">

File: faucon_base_desc/description/gps.xacro (robot description, xacro)
@@ -5,5 +5,5 @@
     <parent link="base_link"/>
     <child link="gnss_frame"/>
-    <origin xyz="0.12 0 0.112" rpy="0 0 0"/>
+    <origin xyz="0.0 0 0.35" rpy="0 0 0"/>
   </joint>
   <link name="gnss_frame">

File: faucon_base_desc/description/imu.xacro (robot description, xacro)
@@ -4,5 +4,5 @@
     <parent link="base_link"/>
     <child link="imu_link"/>
-    <origin xyz="0.1 0 0.112" rpy="-0.01 -0.03 -1.52"/>
+    <origin xyz="0.0 0 0.112" rpy="-0.01 -0.03 -1.52"/>
   </joint>
  <link name="imu_link">

File: faucon_base_desc/description/lidar.xacro (robot description, xacro)
@@ -4,5 +4,5 @@
         <parent link="base_link"/>
         <child link="laser_frame"/>
-        <origin xyz="1.25 0 0.35" rpy="0 0.33 0"/>
+        <origin xyz="0.60 0 0.35" rpy="0 0.33 0"/>
     </joint>
     <link name="laser_frame">

File: faucon_base_desc/description/robot_core_control.xacro (robot description, xacro)
@@ -10,5 +10,5 @@
     <xacro:property name="leg_height" value="0.7"/>
     <xacro:property name="leg_mass" value="0.5"/>
-    <xacro:property name="leg_offset_x" value="1.0"/>
+    <xacro:property name="leg_offset_x" value="0.325"/>
     <xacro:property name="leg_offset_y" value="0.5"/>
     <xacro:property name="leg_offset_z" value="0.1"/>
@@ -16,9 +16,9 @@
     <xacro:property name="wheel_thickness" value="0.1"/>
     <xacro:property name="wheel_mass" value="0.5"/>
-    <xacro:property name="wheel_offset_x" value="1.0"/>
+    <xacro:property name="wheel_offset_x" value="0.325"/>
     <xacro:property name="wheel_offset_y" value="0.5"/>
     <xacro:property name="wheel_offset_z" value="0.01"/>
     <xacro:property name="caster_wheel_radius" value="0.12"/>
-    <xacro:property name="caster_wheel_offset_x" value="0.350"/>
+    <xacro:property name="caster_wheel_offset_x" value="-0.325"/>
     <xacro:property name="caster_wheel_offset_z" value="${wheel_offset_z - wheel_radius + caster_wheel_radius}"/>
     <material name="white">
@@ -47,5 +47,5 @@
     <link name="base_link">
         <visual>
-            <origin xyz="${chassis_length/2} 0 ${chassis_height/2}"/>
+            <origin xyz="0 0 ${chassis_height/2}"/>
             <geometry>
                 <box size="${chassis_length} ${chassis_width} ${chassis_height}"/>
@@ -54,5 +54,5 @@
         </visual>
         <collision>
-            <origin xyz="${chassis_length/2} 0 ${chassis_height/2}"/>
+            <origin xyz="0 0 ${chassis_height/2}"/>
             <geometry>
                 <box size="${chassis_length} ${chassis_width} ${chassis_height}"/>
